Commit message: Added bumper controller

File: src/amr_description/urdf/amr_gazebo.xacro (robot description, xacro)
@@ -35,4 +35,7 @@
       </plugin>
       <plugin filename="gz-sim-imu-system" name="gz::sim::systems::Imu">
+      </plugin>
+      <plugin filename="gz-sim-sensors-system" name="gz::sim::systems::Sensors">
+        <render_engine>ogre2</render_engine>
       </plugin>
   </gazebo>
@@ -88,3 +91,32 @@
     </sensor>
   </gazebo>
+  <gazebo reference="Lidar_Link">
+    <sensor name="lidar" type="gpu_lidar">
+      <always_on>true</always_on>
+      <visualize>true</visualize>
+      <topic>/scan</topic>
+      <update_rate>5</update_rate>
+      <gz_frame_id>Lidar_Link</gz_frame_id>
+      <lidar>
+        <scan>
+          <horizontal>
+            <samples>360</samples>
+            <resolution>1.00</resolution>
+            <min_angle>0.00</min_angle>
+            <max_angle>6.28</max_angle>
+          </horizontal>
+        </scan>
+        <range>
+          <min>0.120</min>
+          <max>12.0</max>
+          <resolution>0.02</resolution>
+        </range>
+        <noise>
+          <type>gaussian</type>
+          <mean>0.0</mean>
+          <stddev>0.01</stddev>
+        </noise>
+      </lidar>
+    </sensor>
+  </gazebo>
 </robot>

File: src/amr_description/urdf/amr_ros2_control.xacro (robot description, xacro)
@@ -21,4 +21,22 @@
             <state_interface name="velocity" />
         </joint>
-    </ros2_control>
+    <!-- ADDED: Front Bumper -->
+        <joint name="Front_Bumper_Joint">
+            <command_interface name="position">
+              <param name="min">-0.01</param>
+              <param name="max">0.0</param>
+            </command_interface>
+            <state_interface name="position" />
+            <state_interface name="velocity" />
+        </joint>
+        <!-- ADDED: Rear Bumper -->
+        <joint name="Rear_Bumper_Joint">
+            <command_interface name="position">
+              <param name="min">0.0</param>
+              <param name="max">0.01</param>
+            </command_interface>
+            <state_interface name="position" />
+            <state_interface name="velocity" />
+        </joint>
+   </ros2_control>
 </robot>
