Commit message: Completed till Differential Kinematics

File: src/amr_description/urdf/amr.urdf.xacro (robot description, xacro)
@@ -56,10 +56,9 @@
                        w="${base_width}"
                        h="${base_height}"/>
-                       <visual>
-      <origin
-        xyz="0.06 0 -0.0368"
-        rpy="0 0 -${pi/2}" />
-      <geometry>
-        <!-- <box size="${base_length} ${base_width} ${base_height}"/> -->
+    <visual>
+      <origin
+        xyz="0 0 0"
+        rpy="0 0 0" />
+      <geometry>
         <mesh filename="package://amr_description/meshes/Base_Link.STL" scale="0.001 0.001 0.001"/>
       </geometry>
@@ -74,5 +73,4 @@
         rpy="0 0 0" />
       <geometry>
-        <!-- <box size="0.600 0.500 0.180"/> -->
         <mesh filename="package://amr_description/meshes/Base_Link.STL" scale="0.001 0.001 0.001"/>
       </geometry>
@@ -94,5 +92,4 @@
         rpy="0 0 0" />
       <geometry>
-        <!-- <cylinder radius="${wheel_radius}" length="${wheel_width}"/> -->
         <mesh filename="package://amr_description/meshes/Right_Wheel.STL" scale="0.001 0.001 0.001"/>
       </geometry>
@@ -127,5 +124,4 @@
         rpy="0 0 0" />
       <geometry>
-        <!-- <cylinder radius="${wheel_radius}" length="${wheel_width}"/> -->
         <mesh filename="package://amr_description/meshes/Left_Wheel.STL" scale="0.001 0.001 0.001"/>
       </geometry>
@@ -158,5 +154,4 @@
         rpy="0 0 0" />
       <geometry>
-        <!-- <sphere radius="${caster_radius}"/> -->
         <mesh filename="package://amr_description/meshes/Caster.STL" scale="0.001 0.001 0.001" />
       </geometry>
@@ -169,6 +164,5 @@
       <origin xyz="0 0 0" rpy="0 0 0"/>
       <geometry>
-        <sphere radius="0.020"/>
-        <!-- <mesh filename="package://amr_description/meshes/Caster.STL" scale="0.001 0.001 0.001" />  -->
+        <mesh filename="package://amr_description/meshes/Caster.STL" scale="0.001 0.001 0.001" />
       </geometry>
     </collision>
@@ -190,5 +184,4 @@
         rpy="0 0 ${pi}" />
       <geometry>
-        <!-- <cylinder radius="0.04" length="${lidar_z}"/> -->
         <mesh filename="package://amr_description/meshes/Lidar.STL" />
       </geometry>
@@ -202,6 +195,5 @@
       <origin xyz="0 0 0" rpy="0 0 ${pi}"/>
       <geometry>
-        <cylinder radius="0.04" length="0.07"/>
-        <!-- <mesh filename="package://amr_description/meshes/Lidar.STL" /> -->
+        <mesh filename="package://amr_description/meshes/Lidar.STL" />
       </geometry>
     </collision>
@@ -225,5 +217,4 @@
         rpy="0 0 0" />
       <geometry>
-        <!-- <box size="0.02 0.02 0.01"/> -->
         <mesh filename="package://amr_description/meshes/IMU.STL" scale="0.001 0.001 0.001"/>
       </geometry>
@@ -237,6 +228,5 @@
       <origin xyz="0 0 0" rpy="0 0 0"/>
       <geometry>
-        <box size="0.02 0.02 0.01"/>
-        <!-- <mesh filename="package://amr_description/meshes/IMU.STL" scale="0.001 0.001 0.001"/> -->
+        <mesh filename="package://amr_description/meshes/IMU.STL" scale="0.001 0.001 0.001"/>
       </geometry>
     </collision>
@@ -265,5 +255,4 @@
       <origin xyz="0 0 0" rpy="0 0 0" />
       <geometry>
-        <!-- <box size="0.05 0.500 0.050"/> -->
         <mesh filename="package://amr_description/meshes/Front_Bumper.STL" scale="0.001 0.001 0.001"/>
       </geometry>
@@ -275,6 +264,5 @@
       <origin xyz="0 0 0" rpy="0 0 0"/>
       <geometry>
-        <box size="0.05 0.500 0.050"/>
-        <!-- <mesh filename="package://amr_description/meshes/Front_Bumper.STL" scale="0.001 0.001 0.001"/> -->
+        <mesh filename="package://amr_description/meshes/Front_Bumper.STL" scale="0.001 0.001 0.001"/>
       </geometry>
     </collision>
@@ -305,5 +293,4 @@
       <origin xyz="0 0 0" rpy="0 0 0" />
       <geometry>
-        <!-- <box size="0.05 0.500 0.050"/> -->
         <mesh filename="package://amr_description/meshes/Rear_Bumper.STL" scale="0.001 0.001 0.001"/>
       </geometry>
@@ -315,6 +302,5 @@
       <origin xyz="0 0 0" rpy="0 0 0"/>
       <geometry>
-        <box size="0.05 0.500 0.050"/>
-        <!-- <mesh filename="package://amr_description/meshes/Rear_Bumper.STL" scale="0.001 0.001 0.001"/> -->
+        <mesh filename="package://amr_description/meshes/Rear_Bumper.STL" scale="0.001 0.001 0.001"/>
       </geometry>
     </collision>

File: src/amr_description/urdf/amr_gazebo.xacro (robot description, xacro)
@@ -3,19 +3,19 @@
   <!-- Wheels -->
   <gazebo reference="Right_Wheel">
-    <mu1>100000000000000.0</mu1>
-    <mu2>100000000000000.0</mu2>
+    <mu1>10.0</mu1>
+    <mu2>10.0</mu2>
     <kp>1000000.0</kp>
-    <kd>10.0</kd>
+    <kd>1.0</kd>
     <minDepth>0.001</minDepth>
-    <maxVel>0.1</maxVel>
+    <maxVel>1</maxVel>
     <fdir1>1 0 0</fdir1>
   </gazebo>
   <gazebo reference="Left_Wheel">
-    <mu1>100000000000000.0</mu1>
-    <mu2>100000000000000.0</mu2>
+    <mu1>10.0</mu1>
+    <mu2>10.0</mu2>
     <kp>1000000.0</kp>
-    <kd>10.0</kd>
+    <kd>1.0</kd>
     <minDepth>0.001</minDepth>
-    <maxVel>0.1</maxVel>
+    <maxVel>1</maxVel>
     <fdir1>1 0 0</fdir1>
   </gazebo>

Commit message: Completed till Differential Kinematics

File: src/amr_description/urdf/amr.urdf.xacro (robot description, xacro)
@@ -171,5 +171,5 @@
     <parent link="base_link"/>
     <child  link="Caster"/>
-    <origin xyz="0.290 0 -0.051" rpy="0 0 0"/>
+    <origin xyz="0.290 0 -0.041" rpy="0 0 0"/>
   </joint>
 <!-- ==================== Lidar ==================== -->
@@ -240,7 +240,4 @@
   <link name="Front_Bumper">
     <inertial>
-      <origin
-        xyz="-0.0399729782081634 -1.10758140167784E-05 -0.00357788828092272"
-        rpy="0 0 0" />
       <mass value="0.192323065808925" />
       <inertia
@@ -271,5 +268,5 @@
     <parent link="base_link"/>
     <child  link="Front_Bumper"/>
-    <origin xyz="0.265 0.001 -0.035" rpy="0 0 0"/>
+    <origin xyz="0.328 0.00225 -0.008" rpy="0 0 0"/>
     <axis xyz="1 0 0"/>
     <limit lower="-0.01" upper="0" effort="20" velocity="0.1"/>
@@ -278,7 +275,4 @@
   <link name="Rear_Bumper">
     <inertial>
-      <origin
-        xyz="0.0177717440542838 -2.23891763389331E-05 -0.0025941331260234"
-        rpy="0 0 0" />
       <mass value="0.14844816742278" />
       <inertia
@@ -309,5 +303,5 @@
     <parent link="base_link"/>
     <child  link="Rear_Bumper"/>
-    <origin xyz="-0.167 0.001 -0.035" rpy="0 0 0"/>
+    <origin xyz="-0.20413 0.00225 -0.008" rpy="0 0 0"/>
     <axis xyz="1 0 0"/>
     <limit lower="0" upper="0.01" effort="20" velocity="0.1"/>

Commit message: Done Sensor Fusion

File: src/amr_description/urdf/amr.urdf.xacro (robot description, xacro)
@@ -49,5 +49,5 @@
     </inertial>
   </xacro:macro>
-  <link name="Base_Footprint"/>
+  <link name="base_footprint"/>
   <!-- ==================== Base Link ==================== -->
   <link name="base_link">
@@ -78,5 +78,5 @@
   </link>
   <joint name="Base_Footprint_Joint" type="fixed">
-    <parent link="Base_Footprint"/>
+    <parent link="base_footprint"/>
     <child  link="base_link"/>
     <origin xyz="0 0 ${wheel_radius}" rpy="0 0 0"/>

Commit message: Weight Distribution Done

File: src/amr_description/urdf/amr.urdf.xacro (robot description, xacro)
@@ -8,18 +8,18 @@
   <xacro:property name="base_width"    value="0.500"/>
   <xacro:property name="base_height"   value="0.180"/>
-  <xacro:property name="base_mass"     value="25.0"/>
+  <xacro:property name="base_mass"     value="30.0"/>
   <xacro:property name="wheel_radius"     value="0.075"/>
   <xacro:property name="wheel_width"      value="0.050"/>
-  <xacro:property name="wheel_mass"       value="2.5"/>
+  <xacro:property name="wheel_mass"       value="1"/>
   <xacro:property name="wheel_separation" value="0.460"/>
   <xacro:property name="caster_radius"    value="0.020"/>
-  <xacro:property name="caster_mass"      value="0.1"/>
+  <xacro:property name="caster_mass"      value="1"/>
   <xacro:property name="lidar_x"         value="0.08"/>
   <xacro:property name="lidar_y"         value="0.08"/>
   <xacro:property name="lidar_z"         value="0.07"/>
-  <xacro:property name="lidar_mass"         value="0.2075"/>
+  <xacro:property name="lidar_mass"         value="1"/>
   <xacro:property name="imu_x"           value="0.04331"/>
   <xacro:property name="imu_y"           value="0.0"/>
-  <xacro:property name="imu_z"           value="0.090"/>
+  <xacro:property name="imu_z"           value="1"/>
   <xacro:macro name="box_inertia" params="m l w h">
     <inertial>

Commit message: Done

File: src/amr_description/urdf/amr.urdf.xacro (robot description, xacro)
@@ -195,5 +195,6 @@
       <origin xyz="0 0 0" rpy="0 0 ${pi}"/>
       <geometry>
-        <mesh filename="package://amr_description/meshes/Lidar.STL" />
+        <box size="0.100 0.070 0.055"/>
+        <!-- <mesh filename="package://amr_description/meshes/Lidar.STL" /> -->
       </geometry>
     </collision>

Commit message: Done Lidar Safety Stop

File: src/amr_description/urdf/amr.urdf.xacro (robot description, xacro)
@@ -12,5 +12,5 @@
   <xacro:property name="wheel_width"      value="0.050"/>
   <xacro:property name="wheel_mass"       value="1"/>
-  <xacro:property name="wheel_separation" value="0.460"/>
+  <xacro:property name="wheel_separation" value="0.480"/>
   <xacro:property name="caster_radius"    value="0.020"/>
   <xacro:property name="caster_mass"      value="1"/>
@@ -269,5 +269,5 @@
     <parent link="base_link"/>
     <child  link="Front_Bumper"/>
-    <origin xyz="0.328 0.00225 -0.008" rpy="0 0 0"/>
+    <origin xyz="0.323 0.00125 -0.007" rpy="0 0 0"/>
     <axis xyz="1 0 0"/>
     <limit lower="-0.01" upper="0" effort="20" velocity="0.1"/>
@@ -304,5 +304,5 @@
     <parent link="base_link"/>
     <child  link="Rear_Bumper"/>
-    <origin xyz="-0.20413 0.00225 -0.008" rpy="0 0 0"/>
+    <origin xyz="-0.20413 0.00125 -0.007" rpy="0 0 0"/>
     <axis xyz="1 0 0"/>
     <limit lower="0" upper="0.01" effort="20" velocity="0.1"/>

Commit message: Bumper, Lidar, Ultrasonic Done

File: src/amr_description/urdf/amr.urdf.xacro (robot description, xacro)
@@ -269,5 +269,5 @@
     <parent link="base_link"/>
     <child  link="Front_Bumper"/>
-    <origin xyz="0.323 0.00125 -0.007" rpy="0 0 0"/>
+    <origin xyz="0.328 0.00125 -0.007" rpy="0 0 0"/>
     <axis xyz="1 0 0"/>
     <limit lower="-0.01" upper="0" effort="20" velocity="0.1"/>
@@ -304,5 +304,5 @@
     <parent link="base_link"/>
     <child  link="Rear_Bumper"/>
-    <origin xyz="-0.20413 0.00125 -0.007" rpy="0 0 0"/>
+    <origin xyz="-0.20913 0.00125 -0.007" rpy="0 0 0"/>
     <axis xyz="1 0 0"/>
     <limit lower="0" upper="0.01" effort="20" velocity="0.1"/>

Commit message: US_links added

File: src/amr_description/urdf/amr.urdf.xacro (robot description, xacro)
@@ -308,3 +308,87 @@
     <limit lower="0" upper="0.01" effort="20" velocity="0.1"/>
   </joint>
+<!-- ==================== ULTRASONIC SENSORS ==================== -->
+  <!-- Simulation only — real sensors are on STM32 via ethernet    -->
+  <!-- Blue boxes = front sensors, Orange boxes = rear sensors     -->
+  <!-- Adjust xyz origins to match physical sensor positions       -->
+  <!-- Front Left Ultrasonic (index 0) -->
+  <link name="Ultrasonic_FL_Link">
+    <inertial>
+      <mass value="0.01"/>
+      <inertia ixx="0.000001" ixy="0" ixz="0"
+               iyy="0.000001" iyz="0"
+               izz="0.000001"/>
+    </inertial>
+    <visual>
+      <geometry><box size="0.02 0.02 0.02"/></geometry>
+      <material name="ultrasonic_front">
+        <color rgba="0 0 1 1"/>
+      </material>
+    </visual>
+  </link>
+  <joint name="Ultrasonic_FL_Joint" type="fixed">
+    <parent link="base_link"/>
+    <child  link="Ultrasonic_FL_Link"/>
+    <origin xyz="0.300  0.150  0.090" rpy="0 0 0"/>
+  </joint>
+  <!-- Front Right Ultrasonic (index 1) -->
+  <link name="Ultrasonic_FR_Link">
+    <inertial>
+      <mass value="0.01"/>
+      <inertia ixx="0.000001" ixy="0" ixz="0"
+               iyy="0.000001" iyz="0"
+               izz="0.000001"/>
+    </inertial>
+    <visual>
+      <geometry><box size="0.02 0.02 0.02"/></geometry>
+      <material name="ultrasonic_front">
+        <color rgba="0 0 1 1"/>
+      </material>
+    </visual>
+  </link>
+  <joint name="Ultrasonic_FR_Joint" type="fixed">
+    <parent link="base_link"/>
+    <child  link="Ultrasonic_FR_Link"/>
+    <origin xyz="0.300 -0.150  0.090" rpy="0 0 0"/>
+  </joint>
+  <!-- Rear Left Ultrasonic (index 2) -->
+  <link name="Ultrasonic_RL_Link">
+    <inertial>
+      <mass value="0.01"/>
+      <inertia ixx="0.000001" ixy="0" ixz="0"
+               iyy="0.000001" iyz="0"
+               izz="0.000001"/>
+    </inertial>
+    <visual>
+      <geometry><box size="0.02 0.02 0.02"/></geometry>
+      <material name="ultrasonic_rear">
+        <color rgba="1 0.5 0 1"/>
+      </material>
+    </visual>
+  </link>
+  <joint name="Ultrasonic_RL_Joint" type="fixed">
+    <parent link="base_link"/>
+    <child  link="Ultrasonic_RL_Link"/>
+    <origin xyz="-0.200  0.150  0.090" rpy="0 0 ${pi}"/>
+  </joint>
+  <!-- Rear Right Ultrasonic (index 3) -->
+  <link name="Ultrasonic_RR_Link">
+    <inertial>
+      <mass value="0.01"/>
+      <inertia ixx="0.000001" ixy="0" ixz="0"
+               iyy="0.000001" iyz="0"
+               izz="0.000001"/>
+    </inertial>
+    <visual>
+      <geometry><box size="0.02 0.02 0.02"/></geometry>
+      <material name="ultrasonic_rear">
+        <color rgba="1 0.5 0 1"/>
+      </material>
+    </visual>
+  </link>
+  <joint name="Ultrasonic_RR_Joint" type="fixed">
+    <parent link="base_link"/>
+    <child  link="Ultrasonic_RR_Link"/>
+    <origin xyz="-0.200 -0.150  0.090" rpy="0 0 ${pi}"/>
+  </joint>
 </robot>
