Commit message: Ultrasonic

File: src/amr_description/urdf/amr.urdf.xacro (robot description, xacro)
@@ -279,5 +279,4 @@
     <limit lower="0" upper="0.01" effort="20" velocity="0.1"/>
   </joint>
-<<<<<<< HEAD
   <!-- ==================== Ultrasonic 1 ==================== -->
   <link name="Ultrasonic_1">
@@ -289,5 +288,5 @@
       <origin xyz="0 0 0" rpy="0 0 0" />
       <geometry>
-        <mesh filename="package://amr_description/meshes/Ultrasonic.STL" scale="0.001 0.001 0.001"/>
+        <mesh filename="package://amr_description/meshes/Ultrasonic_1.STL"/>
       </geometry>
       <material name="">
@@ -298,5 +297,5 @@
       <origin xyz="0 0 0" rpy="0 0 0"/>
       <geometry>
-        <mesh filename="package://amr_description/meshes/Ultrasonic.STL" scale="0.001 0.001 0.001"/>
+        <mesh filename="package://amr_description/meshes/Ultrasonic_1.STL"/>
       </geometry>
     </collision>
@@ -305,5 +304,5 @@
     <parent link="base_link"/>
     <child  link="Ultrasonic_1"/>
-    <origin xyz="-0.4 0.0 0.01" rpy="0 0 0"/>
+    <origin  xyz="0.326401755379924 0.142760073109966 0.062124192966864" rpy="0 0 0"/>
   </joint>
   <!-- ==================== Ultrasonic 2 ==================== -->
@@ -316,14 +315,14 @@
       <origin xyz="0 0 0" rpy="0 0 0" />
       <geometry>
-        <mesh filename="package://amr_description/meshes/Ultrasonic.STL" scale="0.001 0.001 0.001"/>
-      </geometry>
-      <material name="">
-        <color rgba="1 1 1 1" />
-      </material>
-    </visual>
-    <collision>
-      <origin xyz="0 0 0" rpy="0 0 0"/>
-      <geometry>
-        <mesh filename="package://amr_description/meshes/Ultrasonic.STL" scale="0.001 0.001 0.001"/>
+        <mesh filename="package://amr_description/meshes/Ultrasonic_2.STL"/>
+      </geometry>
+      <material name="">
+        <color rgba="0 0 0 1" />
+      </material>
+    </visual>
+    <collision>
+      <origin xyz="0 0 0" rpy="0 0 0"/>
+      <geometry>
+        <mesh filename="package://amr_description/meshes/Ultrasonic_2.STL"/>
       </geometry>
     </collision>
@@ -332,92 +331,59 @@
     <parent link="base_link"/>
     <child  link="Ultrasonic_2"/>
-    <origin xyz="0.4 0.0 0.01" rpy="0 0 0"/>
+    <origin xyz="0.327164794627501 -0.141331027587016 0.062124192966864" rpy="0 0 0"/>
+  </joint>
+  <!-- ==================== Ultrasonic 3 ==================== -->
+  <link name="Ultrasonic_3">
+    <xacro:box_inertia m="${ultrasonic_mass}"
+                       l="${ultrasonic_length}"
+                       w="${ultrasonic_width}"
+                       h="${ultrasonic_height}"/>
+    <visual>
+      <origin xyz="0 0 0" rpy="0 0 0" />
+      <geometry>
+        <mesh filename="package://amr_description/meshes/Ultrasonic_3.STL"/>
+      </geometry>
+      <material name="">
+        <color rgba="0 0 0 1" />
+      </material>
+    </visual>
+    <collision>
+      <origin xyz="0 0 0" rpy="0 0 0"/>
+      <geometry>
+        <mesh filename="package://amr_description/meshes/Ultrasonic_3.STL"/>
+      </geometry>
+    </collision>
+  </link>
+  <joint name="Ultrasonic_3_Joint" type="fixed">
+    <parent link="base_link"/>
+    <child  link="Ultrasonic_3"/>
+    <origin xyz="-0.207113047596706 -0.14142793170944 0.062124192966864" rpy="0 0 0"/>
+  </joint>
+  <!-- ==================== Ultrasonic 4 ==================== -->
+  <link name="Ultrasonic_4">
+    <xacro:box_inertia m="${ultrasonic_mass}"
+                       l="${ultrasonic_length}"
+                       w="${ultrasonic_width}"
+                       h="${ultrasonic_height}"/>
+    <visual>
+      <origin xyz="0 0 0" rpy="0 0 0" />
+      <geometry>
+        <mesh filename="package://amr_description/meshes/Ultrasonic_4.STL"/>
+      </geometry>
+      <material name="">
+        <color rgba="0 0 0 1" />
+      </material>
+    </visual>
+    <collision>
+      <origin xyz="0 0 0" rpy="0 0 0"/>
+      <geometry>
+        <mesh filename="package://amr_description/meshes/Ultrasonic_4.STL"/>
+      </geometry>
+    </collision>
+  </link>
+  <joint name="Ultrasonic_4_Joint" type="fixed">
+    <parent link="base_link"/>
+    <child  link="Ultrasonic_4"/>
+    <origin xyz="-0.20645349231444 0.142663168987541 0.062124192966864" rpy="0 0 0"/>
   </joint>
 </robot>
-=======
-<!-- ==================== ULTRASONIC SENSORS ==================== -->
-  <!-- Simulation only — real sensors are on STM32 via ethernet    -->
-  <!-- Blue boxes = front sensors, Orange boxes = rear sensors     -->
-  <!-- Adjust xyz origins to match physical sensor positions       -->
-  <!-- Front Left Ultrasonic (index 0) -->
-  <link name="Ultrasonic_FL_Link">
-    <inertial>
-      <mass value="0.01"/>
-      <inertia ixx="0.000001" ixy="0" ixz="0"
-               iyy="0.000001" iyz="0"
-               izz="0.000001"/>
-    </inertial>
-    <visual>
-      <geometry><box size="0.02 0.02 0.02"/></geometry>
-      <material name="ultrasonic_front">
-        <color rgba="0 0 1 1"/>
-      </material>
-    </visual>
-  </link>
-  <joint name="Ultrasonic_FL_Joint" type="fixed">
-    <parent link="base_link"/>
-    <child  link="Ultrasonic_FL_Link"/>
-    <origin xyz="0.300  0.150  0.090" rpy="0 0 0"/>
-  </joint>
-  <!-- Front Right Ultrasonic (index 1) -->
-  <link name="Ultrasonic_FR_Link">
-    <inertial>
-      <mass value="0.01"/>
-      <inertia ixx="0.000001" ixy="0" ixz="0"
-               iyy="0.000001" iyz="0"
-               izz="0.000001"/>
-    </inertial>
-    <visual>
-      <geometry><box size="0.02 0.02 0.02"/></geometry>
-      <material name="ultrasonic_front">
-        <color rgba="0 0 1 1"/>
-      </material>
-    </visual>
-  </link>
-  <joint name="Ultrasonic_FR_Joint" type="fixed">
-    <parent link="base_link"/>
-    <child  link="Ultrasonic_FR_Link"/>
-    <origin xyz="0.300 -0.150  0.090" rpy="0 0 0"/>
-  </joint>
-  <!-- Rear Left Ultrasonic (index 2) -->
-  <link name="Ultrasonic_RL_Link">
-    <inertial>
-      <mass value="0.01"/>
-      <inertia ixx="0.000001" ixy="0" ixz="0"
-               iyy="0.000001" iyz="0"
-               izz="0.000001"/>
-    </inertial>
-    <visual>
-      <geometry><box size="0.02 0.02 0.02"/></geometry>
-      <material name="ultrasonic_rear">
-        <color rgba="1 0.5 0 1"/>
-      </material>
-    </visual>
-  </link>
-  <joint name="Ultrasonic_RL_Joint" type="fixed">
-    <parent link="base_link"/>
-    <child  link="Ultrasonic_RL_Link"/>
-    <origin xyz="-0.200  0.150  0.090" rpy="0 0 ${pi}"/>
-  </joint>
-  <!-- Rear Right Ultrasonic (index 3) -->
-  <link name="Ultrasonic_RR_Link">
-    <inertial>
-      <mass value="0.01"/>
-      <inertia ixx="0.000001" ixy="0" ixz="0"
-               iyy="0.000001" iyz="0"
-               izz="0.000001"/>
-    </inertial>
-    <visual>
-      <geometry><box size="0.02 0.02 0.02"/></geometry>
-      <material name="ultrasonic_rear">
-        <color rgba="1 0.5 0 1"/>
-      </material>
-    </visual>
-  </link>
-  <joint name="Ultrasonic_RR_Joint" type="fixed">
-    <parent link="base_link"/>
-    <child  link="Ultrasonic_RR_Link"/>
-    <origin xyz="-0.200 -0.150  0.090" rpy="0 0 ${pi}"/>
-  </joint>
-</robot>
->>>>>>> e77684513a46a55a4d31b0126a36f1a187dda99b

File: src/amr_description/urdf/amr_gazebo.xacro (robot description, xacro)
@@ -120,34 +120,29 @@
     </sensor>
   </gazebo>
-<!-- ==================== ULTRASONIC SENSOR PLUGINS ==================== -->
-  <!-- Each sensor uses gpu_lidar with 1 sample — identical behaviour     -->
-  <!-- to a real ultrasonic sensor for our distance-threshold purposes.   -->
-  <!-- Topics are individual per sensor; ultrasonic_sim_bridge.py         -->
-  <!-- combines them into /ultrasonic_raw matching the real STM32 output. -->
   <!-- Front Left (index 0) -->
-  <gazebo reference="Ultrasonic_FL_Link">
-    <sensor name="ultrasonic_fl" type="gpu_lidar">
-      <always_on>true</always_on>
-      <update_rate>10</update_rate>
-      <topic>ultrasonic_fl_raw</topic>
-      <gz_frame_id>Ultrasonic_FL_Link</gz_frame_id>
-      <lidar>
-        <scan>
-          <horizontal>
-            <samples>1</samples>
-            <resolution>1</resolution>
-            <min_angle>0</min_angle>
-            <max_angle>0</max_angle>
-          </horizontal>
-          <vertical>
-            <samples>1</samples>
-            <resolution>1</resolution>
-            <min_angle>0</min_angle>
-            <max_angle>0</max_angle>
-          </vertical>
-        </scan>
-        <range>
-          <min>0.030</min>
-          <max>5.000</max>
+  <gazebo reference="Ultrasonic_1">
+    <sensor name="ultrasonic_1" type="gpu_lidar">
+      <always_on>true</always_on>
+      <update_rate>10</update_rate>
+      <topic>/ultrasonic_1_raw</topic>
+      <gz_frame_id>Ultrasonic_1</gz_frame_id>
+      <lidar>
+        <scan>
+          <horizontal>
+            <samples>1</samples>
+            <resolution>1</resolution>
+            <min_angle>0</min_angle>
+            <max_angle>0</max_angle>
+          </horizontal>
+          <vertical>
+            <samples>1</samples>
+            <resolution>1</resolution>
+            <min_angle>0</min_angle>
+            <max_angle>0</max_angle>
+          </vertical>
+        </scan>
+        <range>
+          <min>0.030</min>
+          <max>0.300</max>
           <resolution>0.001</resolution>
         </range>
@@ -156,88 +151,88 @@
   </gazebo>
   <!-- Front Right (index 1) -->
-  <gazebo reference="Ultrasonic_FR_Link">
-    <sensor name="ultrasonic_fr" type="gpu_lidar">
-      <always_on>true</always_on>
-      <update_rate>10</update_rate>
-      <topic>ultrasonic_fr_raw</topic>
-      <gz_frame_id>Ultrasonic_FR_Link</gz_frame_id>
-      <lidar>
-        <scan>
-          <horizontal>
-            <samples>1</samples>
-            <resolution>1</resolution>
-            <min_angle>0</min_angle>
-            <max_angle>0</max_angle>
-          </horizontal>
-          <vertical>
-            <samples>1</samples>
-            <resolution>1</resolution>
-            <min_angle>0</min_angle>
-            <max_angle>0</max_angle>
-          </vertical>
-        </scan>
-        <range>
-          <min>0.030</min>
-          <max>5.000</max>
-          <resolution>0.001</resolution>
-        </range>
-      </lidar>
-    </sensor>
-  </gazebo>
-  <!-- Rear Left (index 2) -->
-  <gazebo reference="Ultrasonic_RL_Link">
-    <sensor name="ultrasonic_rl" type="gpu_lidar">
-      <always_on>true</always_on>
-      <update_rate>10</update_rate>
-      <topic>ultrasonic_rl_raw</topic>
-      <gz_frame_id>Ultrasonic_RL_Link</gz_frame_id>
-      <lidar>
-        <scan>
-          <horizontal>
-            <samples>1</samples>
-            <resolution>1</resolution>
-            <min_angle>0</min_angle>
-            <max_angle>0</max_angle>
-          </horizontal>
-          <vertical>
-            <samples>1</samples>
-            <resolution>1</resolution>
-            <min_angle>0</min_angle>
-            <max_angle>0</max_angle>
-          </vertical>
-        </scan>
-        <range>
-          <min>0.030</min>
-          <max>5.000</max>
-          <resolution>0.001</resolution>
-        </range>
-      </lidar>
-    </sensor>
-  </gazebo>
-  <!-- Rear Right (index 3) -->
-  <gazebo reference="Ultrasonic_RR_Link">
-    <sensor name="ultrasonic_rr" type="gpu_lidar">
-      <always_on>true</always_on>
-      <update_rate>10</update_rate>
-      <topic>ultrasonic_rr_raw</topic>
-      <gz_frame_id>Ultrasonic_RR_Link</gz_frame_id>
-      <lidar>
-        <scan>
-          <horizontal>
-            <samples>1</samples>
-            <resolution>1</resolution>
-            <min_angle>0</min_angle>
-            <max_angle>0</max_angle>
-          </horizontal>
-          <vertical>
-            <samples>1</samples>
-            <resolution>1</resolution>
-            <min_angle>0</min_angle>
-            <max_angle>0</max_angle>
-          </vertical>
-        </scan>
-        <range>
-          <min>0.030</min>
-          <max>5.000</max>
+  <gazebo reference="Ultrasonic_2">
+    <sensor name="ultrasonic_2" type="gpu_lidar">
+      <always_on>true</always_on>
+      <update_rate>10</update_rate>
+      <topic>/ultrasonic_2_raw</topic>
+      <gz_frame_id>Ultrasonic_2</gz_frame_id>
+      <lidar>
+        <scan>
+          <horizontal>
+            <samples>1</samples>
+            <resolution>1</resolution>
+            <min_angle>0</min_angle>
+            <max_angle>0</max_angle>
+          </horizontal>
+          <vertical>
+            <samples>1</samples>
+            <resolution>1</resolution>
+            <min_angle>0</min_angle>
+            <max_angle>0</max_angle>
+          </vertical>
+        </scan>
+        <range>
+          <min>0.030</min>
+          <max>0.300</max>
+          <resolution>0.001</resolution>
+        </range>
+      </lidar>
+    </sensor>
+  </gazebo>
+  <!-- Rear Right (index 2) -->
+  <gazebo reference="Ultrasonic_3">
+    <sensor name="ultrasonic_3" type="gpu_lidar">
+      <always_on>true</always_on>
+      <update_rate>10</update_rate>
+      <topic>/ultrasonic_3_raw</topic>
+      <gz_frame_id>Ultrasonic_3</gz_frame_id>
+      <lidar>
+        <scan>
+          <horizontal>
+            <samples>1</samples>
+            <resolution>1</resolution>
+            <min_angle>0</min_angle>
+            <max_angle>0</max_angle>
+          </horizontal>
+          <vertical>
+            <samples>1</samples>
+            <resolution>1</resolution>
+            <min_angle>0</min_angle>
+            <max_angle>0</max_angle>
+          </vertical>
+        </scan>
+        <range>
+          <min>0.030</min>
+          <max>0.200</max>
+          <resolution>0.001</resolution>
+        </range>
+      </lidar>
+    </sensor>
+  </gazebo>
+  <!-- Rear Left (index 3) -->
+  <gazebo reference="Ultrasonic_4">
+    <sensor name="ultrasonic_4" type="gpu_lidar">
+      <always_on>true</always_on>
+      <update_rate>10</update_rate>
+      <topic>/ultrasonic_4_raw</topic>
+      <gz_frame_id>Ultrasonic_4</gz_frame_id>
+      <lidar>
+        <scan>
+          <horizontal>
+            <samples>1</samples>
+            <resolution>1</resolution>
+            <min_angle>0</min_angle>
+            <max_angle>0</max_angle>
+          </horizontal>
+          <vertical>
+            <samples>1</samples>
+            <resolution>1</resolution>
+            <min_angle>0</min_angle>
+            <max_angle>0</max_angle>
+          </vertical>
+        </scan>
+        <range>
+          <min>0.030</min>
+          <max>0.200</max>
           <resolution>0.001</resolution>
         </range>

Commit message: All Safety features working

File: src/amr_description/urdf/amr.urdf.xacro (robot description, xacro)
@@ -304,5 +304,5 @@
     <parent link="base_link"/>
     <child  link="Ultrasonic_1"/>
-    <origin  xyz="0.326401755379924 0.142760073109966 0.062124192966864" rpy="0 0 0"/>
+    <origin  xyz="0.327 0.1445 0.062124192966864" rpy="0 0 0"/>
   </joint>
   <!-- ==================== Ultrasonic 2 ==================== -->
@@ -331,5 +331,5 @@
     <parent link="base_link"/>
     <child  link="Ultrasonic_2"/>
-    <origin xyz="0.327164794627501 -0.141331027587016 0.062124192966864" rpy="0 0 0"/>
+    <origin xyz="0.3277 -0.1405 0.062124192966864" rpy="0 0 0"/>
   </joint>
   <!-- ==================== Ultrasonic 3 ==================== -->
@@ -358,5 +358,5 @@
     <parent link="base_link"/>
     <child  link="Ultrasonic_3"/>
-    <origin xyz="-0.207113047596706 -0.14142793170944 0.062124192966864" rpy="0 0 0"/>
+    <origin xyz="-0.208 -0.140 0.062124192966864" rpy="0 0 0"/>
   </joint>
   <!-- ==================== Ultrasonic 4 ==================== -->
@@ -385,5 +385,32 @@
     <parent link="base_link"/>
     <child  link="Ultrasonic_4"/>
-    <origin xyz="-0.20645349231444 0.142663168987541 0.062124192966864" rpy="0 0 0"/>
+    <origin xyz="-0.207 0.144 0.062124192966864" rpy="0 0 0"/>
+  </joint>
+  <!-- ==================== Ultrasonic 5 ==================== -->
+  <link name="Ultrasonic_5">
+    <xacro:box_inertia m="${ultrasonic_mass}"
+                       l="${ultrasonic_length}"
+                       w="${ultrasonic_width}"
+                       h="${ultrasonic_height}"/>
+    <visual>
+      <origin xyz="0 0 0" rpy="0 0 -2.652" />
+      <geometry>
+        <mesh filename="package://amr_description/meshes/Ultrasonic_4.STL"/>
+      </geometry>
+      <material name="">
+        <color rgba="0 0 0 1" />
+      </material>
+    </visual>
+    <collision>
+      <origin xyz="0 0 0" rpy="0 0 -2.652"/>
+      <geometry>
+        <mesh filename="package://amr_description/meshes/Ultrasonic_4.STL"/>
+      </geometry>
+    </collision>
+  </link>
+  <joint name="Ultrasonic_5_Joint" type="fixed">
+    <parent link="base_link"/>
+    <child  link="Ultrasonic_5"/>
+    <origin xyz="-0.245 0 0.062124192966864" rpy="0 0 3.14159"/>
   </joint>
 </robot>

File: src/amr_description/urdf/amr_gazebo.xacro (robot description, xacro)
@@ -130,19 +130,19 @@
         <scan>
           <horizontal>
-            <samples>1</samples>
-            <resolution>1</resolution>
-            <min_angle>0</min_angle>
-            <max_angle>0</max_angle>
-          </horizontal>
-          <vertical>
-            <samples>1</samples>
-            <resolution>1</resolution>
-            <min_angle>0</min_angle>
-            <max_angle>0</max_angle>
-          </vertical>
-        </scan>
-        <range>
-          <min>0.030</min>
-          <max>0.300</max>
+            <samples>40</samples>
+            <resolution>1</resolution>
+            <min_angle>0.139</min_angle>
+            <max_angle>0.837</max_angle>
+          </horizontal>
+          <vertical>
+            <samples>1</samples>
+            <resolution>1</resolution>
+            <min_angle>0</min_angle>
+            <max_angle>0</max_angle>
+          </vertical>
+        </scan>
+        <range>
+          <min>0.030</min>
+          <max>0.500</max>
           <resolution>0.001</resolution>
         </range>
@@ -160,19 +160,19 @@
         <scan>
           <horizontal>
-            <samples>1</samples>
-            <resolution>1</resolution>
-            <min_angle>0</min_angle>
-            <max_angle>0</max_angle>
-          </horizontal>
-          <vertical>
-            <samples>1</samples>
-            <resolution>1</resolution>
-            <min_angle>0</min_angle>
-            <max_angle>0</max_angle>
-          </vertical>
-        </scan>
-        <range>
-          <min>0.030</min>
-          <max>0.300</max>
+            <samples>40</samples>
+            <resolution>1</resolution>
+            <min_angle>-0.837</min_angle>
+            <max_angle>-0.139</max_angle>
+          </horizontal>
+          <vertical>
+            <samples>1</samples>
+            <resolution>1</resolution>
+            <min_angle>0</min_angle>
+            <max_angle>0</max_angle>
+          </vertical>
+        </scan>
+        <range>
+          <min>0.030</min>
+          <max>0.500</max>
           <resolution>0.001</resolution>
         </range>
@@ -190,19 +190,19 @@
         <scan>
           <horizontal>
-            <samples>1</samples>
-            <resolution>1</resolution>
-            <min_angle>0</min_angle>
-            <max_angle>0</max_angle>
-          </horizontal>
-          <vertical>
-            <samples>1</samples>
-            <resolution>1</resolution>
-            <min_angle>0</min_angle>
-            <max_angle>0</max_angle>
-          </vertical>
-        </scan>
-        <range>
-          <min>0.030</min>
-          <max>0.200</max>
+            <samples>40</samples>
+            <resolution>1</resolution>
+            <min_angle>-3.0</min_angle>
+            <max_angle>-2.3</max_angle>
+          </horizontal>
+          <vertical>
+            <samples>1</samples>
+            <resolution>1</resolution>
+            <min_angle>0</min_angle>
+            <max_angle>0</max_angle>
+          </vertical>
+        </scan>
+        <range>
+          <min>0.030</min>
+          <max>0.500</max>
           <resolution>0.001</resolution>
         </range>
@@ -220,19 +220,49 @@
         <scan>
           <horizontal>
-            <samples>1</samples>
-            <resolution>1</resolution>
-            <min_angle>0</min_angle>
-            <max_angle>0</max_angle>
-          </horizontal>
-          <vertical>
-            <samples>1</samples>
-            <resolution>1</resolution>
-            <min_angle>0</min_angle>
-            <max_angle>0</max_angle>
-          </vertical>
-        </scan>
-        <range>
-          <min>0.030</min>
-          <max>0.200</max>
+            <samples>40</samples>
+            <resolution>1</resolution>
+            <min_angle>2.3</min_angle>
+            <max_angle>3.0</max_angle>
+          </horizontal>
+          <vertical>
+            <samples>1</samples>
+            <resolution>1</resolution>
+            <min_angle>0</min_angle>
+            <max_angle>0</max_angle>
+          </vertical>
+        </scan>
+        <range>
+          <min>0.030</min>
+          <max>0.500</max>
+          <resolution>0.001</resolution>
+        </range>
+      </lidar>
+    </sensor>
+  </gazebo>
+    <!-- Rear Middle (index 4) -->
+  <gazebo reference="Ultrasonic_5">
+    <sensor name="ultrasonic_5" type="gpu_lidar">
+      <always_on>true</always_on>
+      <update_rate>10</update_rate>
+      <topic>/ultrasonic_5_raw</topic>
+      <gz_frame_id>Ultrasonic_5</gz_frame_id>
+      <lidar>
+        <scan>
+          <horizontal>
+            <samples>40</samples>
+            <resolution>1</resolution>
+            <min_angle>-0.349</min_angle>
+            <max_angle>0.349</max_angle>
+          </horizontal>
+          <vertical>
+            <samples>1</samples>
+            <resolution>1</resolution>
+            <min_angle>0</min_angle>
+            <max_angle>0</max_angle>
+          </vertical>
+        </scan>
+        <range>
+          <min>0.030</min>
+          <max>0.500</max>
           <resolution>0.001</resolution>
         </range>
